File: KiCAD-design-files/board.kicad_pcb (KiCad board)
At the start: 2 copper layers, 37 x 66 mm, 93 parts, among them IC1 TPS61025, P1 CONN_01X04, SW1 FLASH, SW2 RESET, SW3 M_DRV, U1 ESP8266-ESP-03, U2 TPL5111, U3 MCP3021, U4 HDC1080, U5 LPS25HB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

Commit message: Some improvements during first manufacturing
Parts:
- added JP2: JUMPER, footprints:SJ_OPEN, F.Cu at (158.1, 143.2)
- BT1, BT2: value Battery -> 1015
- C2: footprint footprints:C_0805 -> footprints:C_0603
- C3: value 100uF -> DNP
- D1: value Hearthbeat -> LTST-C170KFKT
- D2: value PWR -> LTST-C171KRKT
- L1: footprint footprints:Tayo_Yuden_NR40xx -> footprints:Inductor_1210
- SW1: value FLASH -> PTS820 J15M SMTR LFS; footprint footprints:push-button-SMD-3.7x6.0 -> footprints:Tact_Switch_Top_PTS820
- SW2: value RESET -> PTS820 J15M SMTR LFS; footprint footprints:push-button-SMD-3.7x6.0 -> footprints:Tact_Switch_Top_PTS820
- SW3: value M_DRV -> PTS820 J15M SMTR LFS
- moved SW1 0.51 mm to (155.8, 122.1), turned to 180 degrees
- moved SW2 0.51 mm to (155.8, 109.9), turned to 180 degrees
- moved L1 0.30 mm to (165.0, 136.7)
- moved C2 0.17 mm to (159.8, 133.2)
Routing:
- net +3V3: track 193.3 -> 197.5 mm
- net /SDA: track 89.8 -> 88.4 mm
- net +BATT: track 45.8 -> 45.1 mm
Other:
- rule pad_to_mask_clearance: 0.07 -> 0.13
- board text added: "2016, Nov. @hamityanik"
- board text removed: "2016, Nov. M. Hamit YANIK"

Commit message: Some improvements & 3D CAD files added
Parts:
- C11: value 100uF -> DNP
- C3: value DNP -> 100uF
- D1: value LTST-C170KFKT -> LTST-C170KRKT
- D2: value LTST-C171KRKT -> LTST-C170KRKT
Routing:
- net GND: track 25.1 -> 31.7 mm
- net /SCL: track 96.3 -> 101.1 mm
- net /LOWBATT: track 28.7 -> 30.0 mm
