File: KiCAD-design-files/board.sch (KiCad schematic (older format))
At the start: 62 parts, among them IC1 TPS61025, P1 CONN_01X04, SW1 FLASH, SW2 RESET, SW3 M_DRV, U1 ESP8266-ESP-03, U2 TPL5111, U3 MCP3021, U4 HDC1080, U5 LPS25HB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

Commit message: Some improvements during first manufacturing
Parts:
- added JP2: JUMPER, footprints:SJ_OPEN, symbol Jumper_NO_Small
- BT1: value Battery -> 1015; kicost:ignore (none) -> false
- BT2: value Battery -> 1015
- C2: footprint footprints:C_0805 -> footprints:C_0603; kicost:Desc CAP CER 2.2UF 10V X7R 0805 -> CAP CER 2.2UF 10V X5R 0603; kicost:Manf# GRM21BR71A225KA01L -> GRM188R61A225KE34J
- C3: value 100uF -> DNP; kicost:Desc CAP TANT 100UF 6.3V 20% 1411 -> (none); kicost:Manf AVX Corporation -> (none); kicost:Manf# F930J107MBA -> (none)
- D1: value Hearthbeat -> LTST-C170KRKT; kicost:Desc LED ORANGE CLEAR 0805 SMD -> LED RED CLEAR 0805 SMD; kicost:Manf# LTST-C170KFKT -> LTST-C170KRKT
- D2: value PWR -> LTST-C170KRKT; kicost:Manf# LTST-C171KRKT -> LTST-C170KRKT
- SW1: value FLASH -> PTS820 J15M SMTR LFS; footprint footprints:push-button-SMD-3.7x6.0 -> footprints:Tact_Switch_Top_PTS820; kicost:Manf# RS-282G05A3-SM RT -> PTS820 J15M SMTR LFS; kicost:ignore (none) -> false
- SW2: value RESET -> PTS820 J15M SMTR LFS; footprint footprints:push-button-SMD-3.7x6.0 -> footprints:Tact_Switch_Top_PTS820; kicost:Manf# RS-282G05A3-SM RT -> PTS820 J15M SMTR LFS; kicost:ignore (none) -> false
- SW3: value M_DRV -> PTS820 J15M SMTR LFS; kicost:ignore (none) -> false
Connections:
- net +3V3: now also JP2.1, JP2.2
Other:
- note added: "AA Batteries"
- note added: "FLASH"
- note added: "Hearthbeat"
- note added: "RESET"
- moved on the sheet: D2, R20
Changed lines of the file:
@@
 EESchema Schematic File Version 2
 LIBS:library
+LIBS:board-cache
 EELAYER 25 0
 EELAYER END
@@
 F 0 "C2" H 7910 1920 50  0000 L CNN
 F 1 "2.2uF" H 7910 1770 50  0000 L CNN
-F 2 "footprints:C_0805" H 7900 1850 50  0001 C CNN
+F 2 "footprints:C_0603" H 7900 1850 50  0001 C CNN
 F 3 "" H 7900 1850 50  0000 C CNN
 F 4 "Murata Electronics" H 7900 1850 60  0001 C CNN "kicost:Manf"
-F 5 "GRM21BR71A225KA01L" H 7900 1850 60  0001 C CNN "kicost:Manf#"
-F 6 "CAP CER 2.2UF 10V X7R 0805" H 7900 1850 60  0001 C CNN "kicost:Desc"
+F 5 "GRM188R61A225KE34J" H 7900 1850 60  0001 C CNN "kicost:Manf#"
+F 6 "CAP CER 2.2UF 10V X5R 0603" H 7900 1850 60  0001 C CNN "kicost:Desc"
 F 7 "false" H 7900 1850 60  0001 C CNN "kicost:ignore"
 	1    7900 1850
@@
 P 950 1700
 F 0 "BT1" H 1050 1750 50  0000 L CNN
-F 1 "Battery" H 1050 1650 50  0000 L CNN
+F 1 "1015" H 1050 1650 50  0000 L CNN
 F 2 "footprints:Keystone_1015_Holder_Battery_AA" V 950 1740 50  0001 C CNN
 F 3 "" V 950 1740 50  0000 C CNN
@@
 F 5 "1015" H 950 1700 60  0001 C CNN "kicost:Manf#"
 F 6 "HOLDER BATTERY AA" H 950 1700 60  0001 C CNN "kicost:Desc"
+F 7 "false" H 950 1700 60  0001 C CNN "kicost:ignore"
 	1    950  1700
 	1    0    0    -1
@@
 P 8200 1850
 F 0 "C3" H 8210 1920 50  0000 L CNN
-F 1 "100uF" H 8210 1770 50  0000 L CNN
+F 1 "DNP" H 8210 1770 50  0000 L CNN
 F 2 "footprints:TantalC_SizeB_EIA-3528_Reflow" H 8200 1850 50  0001 C CNN
 F 3 "" H 8200 1850 50  0000 C CNN
-F 4 "AVX Corporation" H 8200 1850 60  0001 C CNN "kicost:Manf"
-F 5 "F930J107MBA" H 8200 1850 60  0001 C CNN "kicost:Manf#"
-F 6 "CAP TANT 100UF 6.3V 20% 1411" H 8200 1850 60  0001 C CNN "kicost:Desc"
-F 7 "false" H 8200 1850 60  0001 C CNN "kicost:ignore"
+F 4 "false" H 8200 1850 60  0001 C CNN "kicost:ignore"
 	1    8200 1850
 	1    0    0    -1
@@
 P 3800 5250
 F 0 "SW2" H 3950 5360 50  0000 C CNN
-F 1 "RESET" H 3800 5170 50  0000 C CNN
-F 2 "footprints:push-button-SMD-3.7x6.0" H 3800 5250 50  0001 C CNN
+F 1 "PTS820 J15M SMTR LFS" H 3950 5150 50  0000 C CNN
+F 2 "footprints:Tact_Switch_Top_PTS820" H 3800 5250 50  0001 C CNN
 F 3 "" H 3800 5250 50  0000 C CNN
 F 4 "C&K" H 3800 5250 60  0001 C CNN "kicost:Manf"
-F 5 "RS-282G05A3-SM RT" H 3800 5250 60  0001 C CNN "kicost:Manf#"
+F 5 "PTS820 J15M SMTR LFS" H 3800 5250 60  0001 C CNN "kicost:Manf#"
 F 6 "SWITCH TACTILE SPST-NO 0.05A 12V" H 3800 5250 60  0001 C CNN "kicost:Desc"
+F 7 "false" H 3800 5250 60  0001 C CNN "kicost:ignore"
 	1    3800 5250
 	1    0    0    -1
@@
 P 3800 4650
 F 0 "SW1" H 3950 4760 50  0000 C CNN
-F 1 "FLASH" H 3800 4570 50  0000 C CNN
-F 2 "footprints:push-button-SMD-3.7x6.0" H 3800 4650 50  0001 C CNN
+F 1 "PTS820 J15M SMTR LFS" H 3950 4550 50  0000 C CNN
+F 2 "footprints:Tact_Switch_Top_PTS820" H 3800 4650 50  0001 C CNN
 F 3 "" H 3800 4650 50  0000 C CNN
 F 4 "C&K" H 3800 4650 60  0001 C CNN "kicost:Manf"
-F 5 "RS-282G05A3-SM RT" H 3800 4650 60  0001 C CNN "kicost:Manf#"
+F 5 "PTS820 J15M SMTR LFS" H 3800 4650 60  0001 C CNN "kicost:Manf#"
 F 6 "SWITCH TACTILE SPST-NO 0.05A 12V" H 3800 4650 60  0001 C CNN "kicost:Desc"
+F 7 "false" H 3800 4650 60  0001 C CNN "kicost:ignore"
 	1    3800 4650
 	1    0    0    -1
@@
 P 950 2050
 F 0 "BT2" H 1050 2100 50  0000 L CNN
-F 1 "Battery" H 1050 2000 50  0000 L CNN
+F 1 "1015" H 1050 2000 50  0000 L CNN
 F 2 "footprints:Keystone_1015_Holder_Battery_AA" V 950 2090 50  0001 C CNN
 F 3 "" V 950 2090 50  0000 C CNN
@@
 P 1150 6750
 F 0 "D1" H 1100 6875 50  0000 L CNN
-F 1 "Hearthbeat" H 975 6650 50  0000 L CNN
+F 1 "LTST-C170KRKT" H 975 6650 50  0000 L CNN
 F 2 "footprints:LED_0805" V 1150 6750 50  0001 C CNN
 F 3 "" V 1150 6750 50  0000 C CNN
 F 4 "Lite-On Inc." H 1150 6750 60  0001 C CNN "kicost:Manf"
-F 5 "LTST-C170KFKT" H 1150 6750 60  0001 C CNN "kicost:Manf#"
-F 6 "LED ORANGE CLEAR 0805 SMD" H 1150 6750 60  0001 C CNN "kicost:Desc"
+F 5 "LTST-C170KRKT" H 1150 6750 60  0001 C CNN "kicost:Manf#"
+F 6 "LED RED CLEAR 0805 SMD" H 1150 6750 60  0001 C CNN "kicost:Desc"
 F 7 "false" H 1150 6750 60  0001 C CNN "kicost:ignore"
 	1    1150 6750
@@
 P 1400 3300
 F 0 "SW3" H 1550 3410 50  0000 C CNN
-F 1 "M_DRV" H 1400 3220 50  0000 C CNN
+F 1 "PTS820 J15M SMTR LFS" H 1400 3220 50  0000 C CNN
 F 2 "footprints:Tact_Switch_Top_PTS820" H 1400 3300 50  0001 C CNN
 F 3 "" H 1400 3300 50  0000 C CNN
@@
 F 5 "PTS820 J15M SMTR LFS" H 1400 3300 60  0001 C CNN "kicost:Manf#"
 F 6 "SWITCH TACTILE SPST-NO 0.05A 12V" H 1400 3300 60  0001 C CNN "kicost:Desc"
+F 7 "false" H 1400 3300 60  0001 C CNN "kicost:ignore"
 	1    1400 3300
 	1    0    0    -1
@@
 L Led_Small D2
 U 1 1 582AEE7A
-P 8600 1850
-F 0 "D2" H 8550 1975 50  0000 L CNN
-F 1 "PWR" H 8425 1750 50  0000 L CNN
-F 2 "footprints:LED_0805" V 8600 1850 50  0001 C CNN
-F 3 "" V 8600 1850 50  0000 C CNN
-F 4 "Lite-On Inc." H 8600 1850 60  0001 C CNN "kicost:Manf"
-F 5 "LTST-C171KRKT" H 8600 1850 60  0001 C CNN "kicost:Manf#"
-F 6 "LED RED CLEAR 0805 SMD" H 8600 1850 60  0001 C CNN "kicost:Desc"
-F 7 "false" H 8600 1850 60  0001 C CNN "kicost:ignore"
-	1    8600 1850
+P 8600 1900
+F 0 "D2" H 8550 1800 50  0000 L CNN
+F 1 "LTST-C170KRKT" H 8600 2000 50  0000 C CNN
+F 2 "footprints:LED_0805" V 8600 1900 50  0001 C CNN
+F 3 "" V 8600 1900 50  0000 C CNN
+F 4 "Lite-On Inc." H 8600 1900 60  0001 C CNN "kicost:Manf"
+F 5 "LTST-C170KRKT" H 8600 1900 60  0001 C CNN "kicost:Manf#"
+F 6 "LED RED CLEAR 0805 SMD" H 8600 1900 60  0001 C CNN "kicost:Desc"
+F 7 "false" H 8600 1900 60  0001 C CNN "kicost:ignore"
+	1    8600 1900
 	0    -1   -1   0
 $EndComp
@@
 L R_Small R20
 U 1 1 582AEE82
-P 8600 2150
-F 0 "R20" H 8630 2170 50  0000 L CNN
-F 1 "1k" H 8630 2110 50  0000 L CNN
-F 2 "footprints:R_0805" H 8600 2150 50  0001 C CNN
-F 3 "" H 8600 2150 50  0000 C CNN
-F 4 "Yageo" H 8600 2150 60  0001 C CNN "kicost:Manf"
-F 5 "RC0805JR-071KL" H 8600 2150 60  0001 C CNN "kicost:Manf#"
-F 6 "RES SMD 1K OHM 5% 1/8W 0805" H 8600 2150 60  0001 C CNN "kicost:Desc"
-F 7 "false" H 8600 2150 60  0001 C CNN "kicost:ignore"
-	1    8600 2150
+P 8600 2200
+F 0 "R20" H 8630 2220 50  0000 L CNN
+F 1 "1k" H 8630 2160 50  0000 L CNN
+F 2 "footprints:R_0805" H 8600 2200 50  0001 C CNN
+F 3 "" H 8600 2200 50  0000 C CNN
+F 4 "Yageo" H 8600 2200 60  0001 C CNN "kicost:Manf"
+F 5 "RC0805JR-071KL" H 8600 2200 60  0001 C CNN "kicost:Manf#"
+F 6 "RES SMD 1K OHM 5% 1/8W 0805" H 8600 2200 60  0001 C CNN "kicost:Desc"
+F 7 "false" H 8600 2200 60  0001 C CNN "kicost:ignore"
+	1    8600 2200
 	1    0    0    -1
 $EndComp
@@
 	7900 1450 7900 1750
 Wire Wire Line
-	6300 1450 8600 1450
+	6300 1450 8650 1450
 Wire Wire Line
 	4850 1450 4850 1750
@@
 	1700 3300 2100 3300
 Wire Wire Line
-	8600 1950 8600 2050
+	8600 2000 8600 2100
 Wire Wire Line
-	8600 2250 8600 2400
-Wire Wire Line
-	8600 1450 8600 1750
+	8600 2300 8600 2400
 Wire Wire Line
 	4050 6300 3700 6300
@@
 	1    0    0    -1
 $EndComp
+$Comp
+L Jumper_NO_Small JP2
+U 1 1 5884B6E8
+P 8600 1600
+F 0 "JP2" H 8600 1750 50  0000 C CNN
+F 1 "JUMPER" H 8600 1800 50  0000 C CNN
+F 2 "footprints:SJ_OPEN" H 8600 1600 50  0001 C CNN
+F 3 "" H 8600 1600 50  0000 C CNN
+F 4 "false" H 8600 1600 60  0001 C CNN "kicost:ignore"
+	1    8600 1600
+	0    1    1    0
+$EndComp
+Wire Wire Line
+	8600 1450 8600 1500
+Wire Wire Line
+	8600 1700 8600 1800
+Wire Wire Line
+	8600 1750 8650 1750
+Wire Wire Line
+	8650 1750 8650 1450
+Connection ~ 8600 1450
+Connection ~ 8600 1750
+Text Notes 3650 4850 0    60   ~ 0
+FLASH
+Text Notes 3650 5450 0    60   ~ 0
+RESET
+Text Notes 1400 6950 1    60   ~ 0
+Hearthbeat
+Text Notes 1400 2150 1    60   ~ 0
+AA Batteries
 $EndSCHEMATC
